Commit message: chassis

File: description/robot_core.xacro (robot description, xacro)
@@ -15,3 +15,17 @@
     <link name='base_link'>
     </link>
+    <joint name="chassis_joint" type='fixed'>
+        <parent link='base_link' />
+        <child link='chassis' />
+        <origin xyz='-0.1 0 0' />
+    </joint>
+    <link name="shassis">
+        <visual>
+            <origin xyz='0.15 0 0.075' />
+            <geometry>
+                <box size="0.3 0.3 0.15" />
+            </geometry>
+            <material name="white" />
+        </visual>
+    </link>
 </robot>

Commit message: wheels

File: description/robot_core.xacro (robot description, xacro)
@@ -13,6 +13,8 @@
         <color rgba="0 0 0 1" />
     </material>
+    <!-- BASE LINK  -->
     <link name='base_link'>
     </link>
+    <!-- CHASSIS LINK -->
     <joint name="chassis_joint" type='fixed'>
         <parent link='base_link' />
@@ -20,5 +22,5 @@
         <origin xyz='-0.1 0 0' />
     </joint>
-    <link name="shassis">
+    <link name="chassis">
         <visual>
             <origin xyz='0.15 0 0.075' />
@@ -29,3 +31,33 @@
         </visual>
     </link>
+    <!-- left wheel -->
+    <joint name='left_wheel_joint' type='continuous'>
+        <parent link='base_link' />
+        <child link='left_wheel' />
+        <origin xyz='0 0.175 0' rpy='-${pi/2} 0 0' />
+        <axis xyz='0 0 1' />
+    </joint>
+    <link name='left_wheel'>
+        <visual>
+            <geometry>
+                <cylinder radius='0.05' length='0.04' />
+            </geometry>
+            <material name='blue' />
+        </visual>
+    </link>
+    <!-- right wheel -->
+    <joint name='right_wheel_joint' type='continuous'>
+        <parent link='base_link' />
+        <child link='right_wheel' />
+        <origin xyz='0 -0.175 0' rpy='${pi/2} 0 0' />
+        <axis xyz='0 0 -1' />
+    </joint>
+    <link name='right_wheel'>
+        <visual>
+            <geometry>
+                <cylinder radius='0.05' length='0.04' />
+            </geometry>
+            <material name='blue' />
+        </visual>
+    </link>
 </robot>

Commit message: added stuff

File: description/robot_core.xacro (robot description, xacro)
@@ -61,3 +61,17 @@
         </visual>
     </link>
+    <!-- caster wheel -->
+    <joint name='caster_wheel_joint' type='fixed'>
+        <parent link='base_link' />
+        <child link='caster_wheel' />
+        <origin xyz='0.25 0 0' />
+    </joint>
+    <link name='caster_wheel'>
+        <visual>
+            <geometry>
+                <sphere radius='0.05' />
+            </geometry>
+            <material name='black' />
+        </visual>
+    </link>
 </robot>

Commit message: added stuff

File: description/robot_core.xacro (robot description, xacro)
@@ -30,4 +30,9 @@
             <material name="white" />
         </visual>
+        <collision>
+            <geometry>
+                <box size="0.3 0.3 0.15" />
+            </geometry>
+        </collision>
     </link>
     <!-- left wheel -->
@@ -45,4 +50,9 @@
             <material name='blue' />
         </visual>
+        <collision>
+            <geometry>
+                <box size="0.3 0.3 0.15" />
+            </geometry>
+        </collision>
     </link>
     <!-- right wheel -->
@@ -60,4 +70,9 @@
             <material name='blue' />
         </visual>
+        <collision>
+            <geometry>
+                <box size="0.3 0.3 0.15" />
+            </geometry>
+        </collision>
     </link>
     <!-- caster wheel -->
@@ -65,5 +80,5 @@
         <parent link='base_link' />
         <child link='caster_wheel' />
-        <origin xyz='0.25 0 0' />
+        <origin xyz='0.24 0 0' />
     </joint>
     <link name='caster_wheel'>
@@ -74,4 +89,9 @@
             <material name='black' />
         </visual>
+        <collision>
+            <geometry>
+                <box size="0.3 0.3 0.15" />
+            </geometry>
+        </collision>
     </link>
 </robot>

Commit message: added stuff

File: description/robot_core.xacro (robot description, xacro)
@@ -1,4 +1,5 @@
 <?xml version="1.0"?>
 <robot xmlns:xacro="http://www.ros.org/wiki/xacro">
+    <xacro:include fileame='inertial_macros.xacro' />
     <material name='white'>
         <color rgba="1 1 1 1" />
@@ -32,7 +33,11 @@
         <collision>
             <geometry>
+                <origin xyz='0.15 0 0.075' />
                 <box size="0.3 0.3 0.15" />
             </geometry>
         </collision>
+        <xacro:inertial_box mass='0.5' x='0.3' y='0.3' z='0.15'>
+            <origin xyz='0.15 0 0.075' rpy='0 0 0' />
+        </xacro:inertial_box>
     </link>
     <!-- left wheel -->
@@ -52,7 +57,10 @@
         <collision>
             <geometry>
-                <box size="0.3 0.3 0.15" />
+                <cylinder radius='0.05' length='0.04' />
             </geometry>
         </collision>
+        <xacro:inertial_cylinder mass='0.1' radius='0.05' length='0.04'>
+            <origin xyz='0 0 0' rpy='0 0 0' />
+        </xacro:inertial_cylinder>
     </link>
     <!-- right wheel -->
@@ -72,7 +80,10 @@
         <collision>
             <geometry>
-                <box size="0.3 0.3 0.15" />
+                <cylinder radius='0.05' length='0.04' />
             </geometry>
         </collision>
+        <xacro:inertial_cylinder mass='0.1' radius='0.05' length='0.04'>
+            <origin xyz='0 0 0' rpy='0 0 0' />
+        </xacro:inertial_cylinder>
     </link>
     <!-- caster wheel -->
@@ -80,5 +91,5 @@
         <parent link='base_link' />
         <child link='caster_wheel' />
-        <origin xyz='0.24 0 0' />
+        <origin xyz='0.20 0 0' />
     </joint>
     <link name='caster_wheel'>
@@ -91,7 +102,10 @@
         <collision>
             <geometry>
-                <box size="0.3 0.3 0.15" />
+                <sphere radius='0.05' />
             </geometry>
         </collision>
+        <xacro:inertial_sphere mass='0.1' radius='0.05'>
+            <origin xyz='0 0 0' rpy='0 0 0' />
+        </xacro:inertial_sphere>
     </link>
 </robot>
